Commit message: Fix vision/TTS auth, cut voice latency, add live self-check and demo video script
Real hardware testing (real camera/mic on the actual dev machine) surfaced
a genuine failure the offline/mocked test suite couldn't catch: object
observation and TTS were calling an experimental interactions.create()
endpoint that this API key gets HTTP 401 on. Both now use the standard,
documented models.generate_content() endpoint (vision.py, tts.py,
gemini_client.py) -- confirmed against the real API (structured vision
returned a synthetic object at (0.71, 0.45); TTS returned a valid WAV).

Also, from that same hardware pass:
- perform_gesture is now NON_BLOCKING so Gemini can start speaking while
  the gesture animation plays, instead of waiting out the whole motion
  first -- cut warm first-audio latency from ~2.2-2.5s to 1.19s measured
  (live_client.py, fsm.py's now-async tool-result handling).
- Removed the ambient scene-memory text nudge entirely: injecting text
  via send_realtime_input always starts a model turn, which raced the
  person's real utterance and caused missing/garbled replies. recall_memory
  already covers the same need on demand.
- Configurable mic RMS threshold (--mic-threshold / CHARACTER_LAMP_MIC_RMS_
  THRESHOLD) plus a rate-limited debug RMS meter in live_capture.py --
  the earlier hardware run showed real engagements but zero completed
  voice turns, which turned out to be a silent threshold mismatch with no
  way to see it.
- New `--check-live`: a hardware-free round trip against the real Gemini
  Live API (connects, answers a BLOCKING tool call, waits for real audio
  + turn_complete) -- lets a demo rehearsal isolate "is it the network/
  model" from "is it the mic/camera" in one command.
- GeminiLiveClient.close() now explicitly closes the websocket instead of
  just joining the thread, and third-party (websocket) logging is capped
  at WARNING so a DEBUG run can't leak the API key via request headers.
- Idle wander is now a small sub-second glance instead of a random
  full-body pose that blocked the attention loop for 3-6s; added missing
  inertial values to the URDF's three fixed semantic links so PyBullet
  stops inventing unit mass for them.
- Silence-to-commit lowered 600ms -> 400ms for a more responsive turn-take.

Updated docs/TECHNICAL_NOTE.md with the real hardware-run measurements
(including the honest "no completed voice turn" finding that drove the
mic-threshold fix) and added docs/DEMO_VIDEO_SCRIPT.md: a timed,
recording-ready shot list with exact dialogue and a post-take checklist
for producing the submission video. 124 tests passing, ruff clean.

Co-Authored-By: Claude Sonnet 5 <noreply@anthropic.com>

File: robot/dummy_lamp_5dof.urdf (robot description, URDF)
Before this commit: robot dummy_character_lamp_5dof, 10 links, 9 joints
Links:
- link camera_link: mass None -> 0.015
- link light_emitter_link: mass None -> 0.010
- link speaker_link: mass None -> 0.005
